Commit message: Make car with 45deg wheels

File: models/gyro-car.urdf (robot description, URDF)
Before this commit: robot faller, 5 links, 4 joints
Links:
- link chassis: mass None -> 10
Joints:
- joint back_left_link: origin xyz=0 0 0 -> xyz=-0.09525 0.06985 0
- joint back_right_link: origin xyz=0 0 0 -> xyz=-0.09525 -0.06985 0
- joint front_left_link: origin xyz=0 0 0 -> xyz=0.09525 0.06985 0
- joint front_right_link: origin xyz=0 0 0 -> xyz=0.09525 -0.06985 0
