Commit message: Add website

File: models/car.urdf (robot description, URDF)
Before this commit: robot faller, 5 links, 4 joints
Joints:
- joint back_left_link: axis 0 1 -1 -> 0 0.7071067812 -0.7071067812; limit (none) -> effort=0 velocity=15000; type continuous -> revolute
- joint back_right_link: axis 0 1 1 -> 0 0.7071067812 0.7071067812; limit (none) -> effort=0 velocity=15000; type continuous -> revolute
- joint front_left_link: axis 0 1 1 -> 0 1 0; limit (none) -> effort=0 velocity=15000; type continuous -> revolute
- joint front_right_link: limit (none) -> effort=0 velocity=15000; type continuous -> revolute
